Commit message: Refactor URDF to use base_link and add base_footprint
Updated link names and joint parents to use 'base_link' instead of 'base'. Added new joint and link for 'base_footprint'.

File: robots/go2w_description/urdf/go2w_description.urdf (robot description, URDF)
Before this commit: robot go2w_description, 33 links, 32 joints
Links:
- removed link base
- removed link radar
- added link base_footprint
- added link base_link, mass 6.921; collision box size=0.3762 0.0935 0.114; visual mesh filename=package://go2w_description/dae/base.dae
- added link utlidar_lidar, mass 0
Joints:
- added joint base_footprint_joint: type fixed, parent base_link, child base_footprint, origin xyz=0 0 -0.05 rpy=0 0 0
- joint FL_hip_joint: parent base -> base_link
- joint FR_hip_joint: parent base -> base_link
- joint Head_upper_joint: parent base -> base_link
- joint RL_hip_joint: parent base -> base_link
- joint RR_hip_joint: parent base -> base_link
- joint imu_joint: parent base -> base_link
- joint radar_joint: child radar -> utlidar_lidar; parent base -> base_link

Commit message: Update mesh file paths to use raw GitHub URLs

File: robots/go2w_description/urdf/go2w_description.urdf (robot description, URDF)
Before this commit: robot go2w_description, 34 links, 33 joints
Links:
- link FL_calf: geometry collision cylinder length=0.12 radius=0.012; visual mesh filename=https://raw.githubusercontent.com/b-dosymzhan/unitree_ros/m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
- link FL_foot: geometry collision mesh filename=https://raw.githubusercontent.com/b-dosymzhan/unitree_ros/m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; visual mesh filename=https://raw.githubusercontent.com/b-dosymzhan/unitree_ros/m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
- link FL_hip: geometry collision cylinder length=0.04 radius=0.046; visual mesh filename=https://raw.githubusercontent.com/b-dosymzhan/unitree_ros/m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
- link FL_thigh: geometry collision box size=0.11 0.0245 0.034; visual mesh filename=https://raw.githubusercontent.com/b-dosymzhan/unitree_ros/m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
- link FR_calf: geometry collision cylinder length=0.12 radius=0.013; visual mesh filename=https://raw.githubusercontent.com/b-dosymzhan/unitree_ros/m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
- link FR_foot: geometry collision mesh filename=https://raw.githubusercontent.com/b-dosymzhan/unitree_ros/m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; visual mesh filename=https://raw.githubusercontent.com/b-dosymzhan/unitree_ros/m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
- link FR_hip: geometry collision cylinder length=0.04 radius=0.046; visual mesh filename=https://raw.githubusercontent.com/b-dosymzhan/unitree_ros/m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
- link FR_thigh: geometry collision box size=0.11 0.0245 0.034; visual mesh filename=https://raw.githubusercontent.com/b-dosymzhan/unitree_ros/m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
- link RL_calf: geometry collision cylinder length=0.12 radius=0.013; visual mesh filename=https://raw.githubusercontent.com/b-dosymzhan/unitree_ros/m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
- link RL_foot: geometry collision mesh filename=https://raw.githubusercontent.com/b-dosymzhan/unitree_ros/m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; visual mesh filename=https://raw.githubusercontent.com/b-dosymzhan/unitree_ros/m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
- link RL_hip: geometry collision cylinder length=0.04 radius=0.046; visual mesh filename=https://raw.githubusercontent.com/b-dosymzhan/unitree_ros/m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
- link RL_thigh: geometry collision box size=0.11 0.0245 0.034; visual mesh filename=https://raw.githubusercontent.com/b-dosymzhan/unitree_ros/m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
- link RR_calf: geometry collision cylinder length=0.12 radius=0.013; visual mesh filename=https://raw.githubusercontent.com/b-dosymzhan/unitree_ros/m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
- link RR_foot: geometry collision mesh filename=https://raw.githubusercontent.com/b-dosymzhan/unitree_ros/m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; visual mesh filename=https://raw.githubusercontent.com/b-dosymzhan/unitree_ros/m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
- link RR_hip: geometry collision cylinder length=0.04 radius=0.046; visual mesh filename=https://raw.githubusercontent.com/b-dosymzhan/unitree_ros/m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
- link RR_thigh: geometry collision box size=0.11 0.0245 0.034; visual mesh filename=https://raw.githubusercontent.com/b-dosymzhan/unitree_ros/m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
- link base_link: geometry collision box size=0.3762 0.0935 0.114; visual mesh filename=https://raw.githubusercontent.com/b-dosymzhan/unitree_ros/m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

Commit message: Update print statement from 'Hello' to 'Goodbye'

File: robots/go2w_description/urdf/go2w_description.urdf (robot description, URDF)
Before this commit: robot go2w_description, 34 links, 33 joints
Links:
- removed link FL_calflower
- removed link FL_calflower1
- removed link FL_foot_motor
- removed link FR_calflower
- removed link FR_calflower1
- removed link FR_foot_motor
- removed link Head_lower
- removed link Head_upper
- removed link RL_calflower
- removed link RL_calflower1
- removed link RL_foot_motor
- removed link RR_calflower
- removed link RR_calflower1
- removed link RR_foot_motor
- removed link imu
- removed link utlidar_lidar
- link FL_calf: mass 0.154 -> None; geometry visual mesh filename=https://raw.githubusercontent.com/b-dosymzhan/unitree_ros/m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
- link FL_foot: mass 0.520 -> None; geometry visual mesh filename=https://raw.githubusercontent.com/b-dosymzhan/unitree_ros/m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
- link FL_hip: mass 0.678 -> None; geometry visual mesh filename=https://raw.githubusercontent.com/b-dosymzhan/unitree_ros/m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
- link FL_thigh: mass 1.152 -> None; geometry visual mesh filename=https://raw.githubusercontent.com/b-dosymzhan/unitree_ros/m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
- link FR_calf: mass 0.154 -> None; geometry visual mesh filename=https://raw.githubusercontent.com/b-dosymzhan/unitree_ros/m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
- link FR_foot: mass 0.520 -> None; geometry visual mesh filename=https://raw.githubusercontent.com/b-dosymzhan/unitree_ros/m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
- link FR_hip: mass 0.678 -> None; geometry visual mesh filename=https://raw.githubusercontent.com/b-dosymzhan/unitree_ros/m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
- link FR_thigh: mass 1.152 -> None; geometry visual mesh filename=https://raw.githubusercontent.com/b-dosymzhan/unitree_ros/m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
- link RL_calf: mass 0.154 -> None; geometry visual mesh filename=https://raw.githubusercontent.com/b-dosymzhan/unitree_ros/m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
- link RL_foot: mass 0.520 -> None; geometry visual mesh filename=https://raw.githubusercontent.com/b-dosymzhan/unitree_ros/m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
- link RL_hip: mass 0.678 -> None; geometry visual mesh filename=https://raw.githubusercontent.com/b-dosymzhan/unitree_ros/m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
- link RL_thigh: mass 1.152 -> None; geometry visual mesh filename=https://raw.githubusercontent.com/b-dosymzhan/unitree_ros/m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
- link RR_calf: mass 0.154 -> None; geometry visual mesh filename=https://raw.githubusercontent.com/b-dosymzhan/unitree_ros/m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
- link RR_foot: mass 0.520 -> None; geometry visual mesh filename=https://raw.githubusercontent.com/b-dosymzhan/unitree_ros/m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
- link RR_hip: mass 0.678 -> None; geometry visual mesh filename=https://raw.githubusercontent.com/b-dosymzhan/unitree_ros/m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
- link RR_thigh: mass 1.152 -> None; geometry visual mesh filename=https://raw.githubusercontent.com/b-dosymzhan/unitree_ros/m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
- link base_link: mass 6.921 -> None; geometry visual mesh filename=https://raw.githubusercontent.com/b-dosymzhan/unitree_ros/m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
Joints:
- removed joint FL_calflower1_joint
- removed joint FL_calflower_joint
- removed joint FL_foot_motor_joint
- removed joint FR_calflower1_joint
- removed joint FR_calflower_joint
- removed joint FR_foot_motor_joint
- removed joint Head_lower_joint
- removed joint Head_upper_joint
- removed joint RL_calflower1_joint
- removed joint RL_calflower_joint
- removed joint RL_foot_motor_joint
- removed joint RR_calflower1_joint
- removed joint RR_calflower_joint
- removed joint RR_foot_motor_joint
- removed joint imu_joint
- removed joint radar_joint
- joint FL_calf_joint: axis 0 1 0 -> (none); limit lower=-2.7227 upper=-0.83776 effort=35.55 velocity=20.07 -> (none); origin xyz=0 0 -0.213 rpy=0 0 0 -> xyz=0 0 -0.213; type revolute -> fixed
- joint FL_foot_joint: axis 0 1 0 -> (none); limit effort=23.7 velocity=30.1 -> (none); origin xyz=0 0 -0.2264 rpy=0 0 0 -> xyz=0 0 -0.2264; type continuous -> fixed
- joint FL_hip_joint: axis 1 0 0 -> (none); limit lower=-1.0472 upper=1.0472 effort=23.7 velocity=30.1 -> (none); origin xyz=0.1934 0.0465 0 rpy=0 0 0 -> xyz=0.1934 0.0465 0; type revolute -> fixed
- joint FL_thigh_joint: axis 0 1 0 -> (none); limit lower=-1.5707963267948966 upper=3.4907 effort=23.7 velocity=30.1 -> (none); origin xyz=0 0.0955 0 rpy=0 0 0 -> xyz=0 0 -0.0955; type revolute -> fixed
- joint FR_calf_joint: axis 0 1 0 -> (none); limit lower=-2.7227 upper=-0.83776 effort=35.55 velocity=20.07 -> (none); origin xyz=0 0 -0.213 rpy=0 0 0 -> xyz=0 0 -0.213; type revolute -> fixed
- joint FR_foot_joint: axis 0 1 0 -> (none); limit effort=23.7 velocity=30.1 -> (none); origin xyz=0 0 -0.2264 rpy=0 0 0 -> xyz=0 0 -0.2264; type continuous -> fixed
- joint FR_hip_joint: axis 1 0 0 -> (none); limit lower=-1.0472 upper=1.0472 effort=23.7 velocity=30.1 -> (none); origin xyz=0.1934 -0.0465 0 rpy=0 0 0 -> xyz=0.1934 -0.0465 0; type revolute -> fixed
- joint FR_thigh_joint: axis 0 1 0 -> (none); limit lower=-1.5707963267948966 upper=3.4907 effort=23.7 velocity=30.1 -> (none); origin xyz=0 -0.0955 0 rpy=0 0 0 -> xyz=0 0 -0.0955; type revolute -> fixed
- joint RL_calf_joint: axis 0 1 0 -> (none); limit lower=-2.7227 upper=-0.83776 effort=35.55 velocity=20.07 -> (none); origin xyz=0 0 -0.213 rpy=0 0 0 -> xyz=0 0 -0.213; type revolute -> fixed
- joint RL_foot_joint: axis 0 1 0 -> (none); limit effort=23.7 velocity=30.1 -> (none); origin xyz=0.0 0 -0.2264 rpy=0 0 0 -> xyz=0 0 -0.2264; type continuous -> fixed
- joint RL_hip_joint: axis 1 0 0 -> (none); limit lower=-1.0472 upper=1.0472 effort=23.7 velocity=30.1 -> (none); origin xyz=-0.1934 0.0465 0 rpy=0 0 0 -> xyz=-0.1934 0.0465 0; type revolute -> fixed
- joint RL_thigh_joint: axis 0 1 0 -> (none); limit lower=-0.5236 upper=4.5379 effort=23.7 velocity=30.1 -> (none); origin xyz=0 0.0955 0 rpy=0 0 0 -> xyz=0 0 -0.0955; type revolute -> fixed
- joint RR_calf_joint: axis 0 1 0 -> (none); limit lower=-2.7227 upper=-0.83776 effort=35.55 velocity=20.07 -> (none); origin xyz=0 0 -0.213 rpy=0 0 0 -> xyz=0 0 -0.213; type revolute -> fixed
- joint RR_foot_joint: axis 0 1 0 -> (none); limit effort=23.7 velocity=30.1 -> (none); origin xyz=-0.0 0 -0.2264 rpy=0 0 0 -> xyz=0 0 -0.2264; type continuous -> fixed
- joint RR_hip_joint: axis 1 0 0 -> (none); limit lower=-1.0472 upper=1.0472 effort=23.7 velocity=30.1 -> (none); origin xyz=-0.1934 -0.0465 0 rpy=0 0 0 -> xyz=-0.1934 -0.0465 0; type revolute -> fixed
- joint RR_thigh_joint: axis 0 1 0 -> (none); limit lower=-0.5236 upper=4.5379 effort=23.7 velocity=30.1 -> (none); origin xyz=0 -0.0955 0 rpy=0 0 0 -> xyz=0 0 -0.0955; type revolute -> fixed
- joint base_footprint_joint: origin xyz=0 0 -0.05 rpy=0 0 0 -> xyz=0 0 -0.05

Commit message: Update go2w_description.urdf

File: robots/go2w_description/urdf/go2w_description.urdf (robot description, URDF)
Before this commit: robot go2w_foxglove, 18 links, 17 joints
Joints:
- joint FL_foot_joint: origin xyz=0 0 -0.2264 -> xyz=0 0 -0.2264 rpy=0 1.5708 1.5708
- joint FR_foot_joint: origin xyz=0 0 -0.2264 -> xyz=0 0 -0.2264 rpy=0 1.5708 1.5708
- joint RL_foot_joint: origin xyz=0 0 -0.2264 -> xyz=0 0 -0.2264 rpy=0 1.5708 1.5708
- joint RR_foot_joint: origin xyz=0 0 -0.2264 -> xyz=0 0 -0.2264 rpy=0 1.5708 1.5708
